Commit message: chore: small changes

File: robot_description/robot.xacro (robot description, xacro)
@@ -48,6 +48,6 @@
   <xacro:property name="camera_inclination" value="${PI/4}"/> <!-- 45° -->
   <!-- Import all Gazebo-customization elements, including Gazebo colors -->
-  <xacro:include filename="$(find exoskeleton)/urdf/robot.gazebo" />
-  <xacro:include filename="$(find exoskeleton)/urdf/realsense_d435.xacro"/>
+  <xacro:include filename="$(find exoskeleton)/robot_description/robot.gazebo" />
+  <xacro:include filename="$(find exoskeleton)/robot_description/realsense_d435.xacro"/>
   <link name="waist_link">
     <collision>
@@ -82,5 +82,5 @@
         <origin xyz="${camera_width} 0 0" rpy="${camera_roll} ${camera_pitch} ${camera_yaw}"/>
             <geometry>
-                <mesh filename="$(find exoskeleton)/urdf/realsense_d435.dae" scale="1 1 1"/>
+                <mesh filename="$(find exoskeleton)/robot_description/realsense_d435.dae" scale="1 1 1"/>
             </geometry>
     </visual>
@@ -88,5 +88,5 @@
         <origin xyz="${camera_width} 0 0" rpy="${camera_roll} ${camera_pitch} ${camera_yaw}"/>
             <geometry>
-                <mesh filename="$(find exoskeleton)/urdf/realsense_d435.dae" scale="1 1 1"/>
+                <mesh filename="$(find exoskeleton)/robot_description/realsense_d435.dae" scale="1 1 1"/>
             </geometry>
         </collision>

Commit message: Update robot.xacro

File: robot_description/robot.xacro (robot description, xacro)
@@ -62,5 +62,7 @@
 	    <box size="${waist_height} ${waist_length} ${waist_width}"/>
       </geometry>
-      <material name="orange"/>
+      <material name="orange">
+        <color rgba="1 0.5 0 1"/>
+      </material>
     </visual>
     <inertial>
@@ -142,5 +144,7 @@
 	    <box size="${up_width} ${up_height} ${up_length}"/>
       </geometry>
-      <material name="orange"/>
+      <material name="orange">
+        <color rgba="1 0.5 0 1"/>
+      </material>
     </visual>
     <inertial>
@@ -174,5 +178,7 @@
 	    <box size="${up_width} ${up_height} ${up_length}"/>
       </geometry>
-      <material name="orange"/>
+      <material name="orange">
+        <color rgba="1 0.5 0 1"/>
+      </material>
     </visual>
     <inertial>
@@ -206,5 +212,7 @@
 	    <box size="${down_width} ${down_height} ${down_length}"/>
       </geometry>
-      <material name="orange"/>
+      <material name="orange">
+        <color rgba="1 0.5 0 1"/>
+      </material>
     </visual>
     <inertial>
@@ -238,5 +246,7 @@
 	    <box size="${down_width} ${down_height} ${down_length}"/>
       </geometry>
-      <material name="orange"/>
+      <material name="orange">
+        <color rgba="1 0.5 0 1"/>
+      </material>
     </visual>
     <inertial>
@@ -273,5 +283,7 @@
 	    <box size="${foot_back_length} ${foot_width} ${foot_height}"/>
       </geometry>
-      <material name="orange"/>
+      <material name="orange">
+        <color rgba="1 0.5 0 1"/>
+      </material>
     </visual>
     <inertial>
@@ -305,5 +317,7 @@
 	    <box size="${foot_back_length} ${foot_width} ${foot_height}"/>
       </geometry>
-      <material name="orange"/>
+      <material name="orange">
+        <color rgba="1 0.5 0 1"/>
+      </material>
     </visual>
     <inertial>
